File: VariablePS.sch (KiCad schematic (older format))
At the start: 18 parts, among them J1 VOUT, J2 VIN, U1 LM317T

Commit message: PCB routing done, gerber files generated (v1.0).
Signed-off-by: Ion Bold <bold.ion86@gmail.com>
Parts:
- C2: footprint Capacitor_THT:CP_Radial_D4.0mm_P2.00mm -> Capacitor_THT:CP_Radial_D5.0mm_P2.50mm
- RV1: footprint (none) -> Potentiometer_THT:Potentiometer_ACP_CA9-H3,8_Horizontal
Changed lines of the file:
@@
 F 0 "C2" H 4568 1796 50  0000 L CNN
 F 1 "2u2" H 4568 1705 50  0000 L CNN
-F 2 "Capacitor_THT:CP_Radial_D4.0mm_P2.00mm" H 4488 1600 50  0001 C CNN
+F 2 "Capacitor_THT:CP_Radial_D5.0mm_P2.50mm" H 4488 1600 50  0001 C CNN
 F 3 "~" H 4450 1750 50  0001 C CNN
 	1    4450 1750
@@
 F 0 "RV1" H 2880 2596 50  0000 R CNN
 F 1 "1k" H 2880 2505 50  0000 R CNN
-F 2 "" H 2950 2550 50  0001 C CNN
+F 2 "Potentiometer_THT:Potentiometer_ACP_CA9-H3,8_Horizontal" H 2950 2550 50  0001 C CNN
 F 3 "~" H 2950 2550 50  0001 C CNN
 	1    2950 2550
